File: afe.kicad_sch (KiCad schematic)
At the start: 0 parts

Commit message: schematic 90%
Parts:
- added C15: 1uF, symbol Device:C
- added C16, C18: 10uF, symbol Device:C
- added C17: 100nF, symbol Device:C
- added U1: MAX86140ENP+T, 21-100134_N201A2-1_MXM, symbol ProjectSymbols:MAX86140ENP+T
Connections:
- new net: C15.2, U1.B5 (VREF)
- new net GND: C15.1, C16.1, C17.2, C18.2, U1.C3 (GND_DIG), U1.C4 (GND_ANA), U1.C5 (PD_GND), U1.D3 (PGND)
- new net GPIO1: U1.B3 (GPIO1)
- new net GPIO2: U1.B4 (GPIO2)
- new net INT: U1.B2 (*INT)
- new net LED1_ANODE: C16.2, U1.A1 (VLED)
- new net LED1_CATHODE: U1.D1 (LED1_DRV)
- new net LED2_CATHODE: U1.C1 (LED2_DRV)
- new net LED3_CATHODE: U1.B1 (LED3_DRV)
- new net PD1: U1.D5 (PD1_IN)
- new net SPI_CSB: U1.A5 (CSB)
- new net SPI_SCLK: U1.A2 (SCLK)
- new net SPI_SDI: U1.A4 (SDI)
- new net SPI_SDO: U1.A3 (SDO)
- new net VDD_ANALOG: C17.1, C18.1, U1.D2 (VDD_ANA)
- new net VDD_DIGITAL: U1.C2 (VDD_DIG)

Commit message: General Structure
Connections:
- net GND: no longer C15.1, U1.C3 (GND_DIG), U1.C4 (GND_ANA), U1.D3 (PGND)
- net LED1_ANODE renamed VDD_LED
- net LED1_CATHODE renamed LED_CATHODE0
- net LED2_CATHODE renamed LED_CATHODE1
- net LED3_CATHODE renamed LED_CATHODE2
- new net ANALOG_GND: C15.1, U1.C3 (GND_DIG), U1.C4 (GND_ANA)
- new net LED_GND: U1.D3 (PGND)
Other:
- company: (none) -> Guardian Health Inc.
- title: (none) -> MAX86140 Analog Front-End

Commit message: inital routing
Parts:
- C15: footprint (none) -> Capacitor_SMD:C_0201_0603Metric
- C16, C17, C18: footprint (none) -> Capacitor_SMD:C_0402_1005Metric
- U1: footprint 21-100134_N201A2-1_MXM -> Project-Symbols:MAX86140ENP+T
Connections:
- net VDD_DIGITAL is gone; now on net VDD_ANALOG: U1.C2 (VDD_DIG)
Other:
- moved on the sheet: C15
Changed lines of the file:
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@@
+	)
+	(junction
+		(at 115.57 55.88)
+		(diameter 0)
+		(color 0 0 0 0)
 	)
 	(junction
@@
 	(wire
 		(pts
-			(xy 88.9 55.88) (xy 118.11 55.88)
+			(xy 88.9 55.88) (xy 115.57 55.88)
 		)
 		(stroke
@@
 	(wire
 		(pts
+			(xy 113.03 66.04) (xy 118.11 66.04)
+		)
+		(stroke
+			(width 0)
+			(type default)
+		)
+	)
+	(wire
+		(pts
 			(xy 184.15 77.47) (xy 185.42 77.47)
 		)
@@
 	(wire
 		(pts
-			(xy 99.06 72.39) (xy 99.06 76.2)
+			(xy 99.06 73.66) (xy 99.06 76.2)
 		)
 		(stroke
@@
 	(wire
 		(pts
+			(xy 115.57 53.34) (xy 115.57 55.88)
+		)
+		(stroke
+			(width 0)
+			(type default)
+		)
+	)
+	(wire
+		(pts
 			(xy 168.91 96.52) (xy 182.88 96.52)
 		)
@@
 	(wire
 		(pts
-			(xy 99.06 64.77) (xy 99.06 60.96)
+			(xy 115.57 53.34) (xy 118.11 53.34)
+		)
+		(stroke
+			(width 0)
+			(type default)
+		)
+	)
+	(wire
+		(pts
+			(xy 99.06 66.04) (xy 99.06 60.96)
 		)
 		(stroke
@@
 		(pts
 			(xy 99.06 76.2) (xy 118.11 76.2)
+		)
+		(stroke
+			(width 0)
+			(type default)
+		)
+	)
+	(wire
+		(pts
+			(xy 115.57 55.88) (xy 118.11 55.88)
 		)
 		(stroke
@@
 	)
 	(hierarchical_label "SPI_SDO"
-		(shape input)
+		(shape output)
 		(at 168.91 55.88 0)
 		(effects
@@
 	)
 	(hierarchical_label "GND"
-		(shape input)
+		(shape passive)
 		(at 88.9 64.77 270)
 		(effects
@@
 	)
 	(hierarchical_label "LED_GND"
-		(shape input)
-		(at 118.11 66.04 180)
+		(shape passive)
+		(at 113.03 66.04 180)
 		(effects
 			(font
@@
 	)
 	(hierarchical_label "GPIO2"
-		(shape input)
+		(shape bidirectional)
 		(at 168.91 69.85 0)
 		(effects
@@
 	)
 	(hierarchical_label "GND"
-		(shape input)
+		(shape passive)
 		(at 76.2 64.77 270)
 		(effects
@@
 	)
 	(hierarchical_label "GND"
-		(shape input)
+		(shape passive)
 		(at 109.22 113.03 180)
 		(effects
@@
 	)
 	(hierarchical_label "INT"
-		(shape input)
+		(shape output)
 		(at 168.91 64.77 0)
 		(effects
@@
 	)
 	(hierarchical_label "ANALOG_GND"
-		(shape input)
+		(shape passive)
 		(at 113.03 63.5 180)
 		(effects
@@
 	)
 	(hierarchical_label "PD_GND"
-		(shape input)
+		(shape passive)
 		(at 109.22 107.95 180)
 		(effects
@@
 	)
 	(hierarchical_label "SPI_SCLK"
-		(shape input)
+		(shape bidirectional)
 		(at 168.91 53.34 0)
 		(effects
@@
 	)
 	(hierarchical_label "GPIO1"
-		(shape input)
+		(shape bidirectional)
 		(at 168.91 67.31 0)
 		(effects
@@
 		)
 	)
-	(hierarchical_label "VDD_DIGITAL"
-		(shape input)
-		(at 118.11 53.34 180)
-		(effects
-			(font
-				(size 1.27 1.27)
-			)
-			(justify right)
-		)
-	)
 	(hierarchical_label "GND"
-		(shape input)
+		(shape passive)
 		(at 171.45 77.47 180)
 		(effects
@@
 	)
 	(hierarchical_label "SPI_CSB"
-		(shape input)
+		(shape bidirectional)
 		(at 168.91 60.96 0)
 		(effects
@@
 			)
 		)
-		(property "Footprint" ""
+		(property "Footprint" "Capacitor_SMD:C_0402_1005Metric"
 			(at 89.8652 63.5 0)
 			(effects
@@
 	(symbol
 		(lib_id "Device:C")
-		(at 99.06 68.58 0)
+		(at 99.06 69.85 0)
 		(unit 1)
 		(exclude_from_sim no)
@@
 		(fields_autoplaced yes)
 		(property "Reference" "C15"
-			(at 102.87 67.3099 0)
+			(at 102.87 68.5799 0)
 			(effects
 				(font
@@
 		)
 		(property "Value" "1uF"
-			(at 102.87 69.8499 0)
+			(at 102.87 71.1199 0)
 			(effects
 				(font
@@
 			)
 		)
-		(property "Footprint" ""
-			(at 100.0252 72.39 0)
+		(property "Footprint" "Capacitor_SMD:C_0201_0603Metric"
+			(at 100.0252 73.66 0)
 			(effects
 				(font
@@
 		)
 		(property "Datasheet" "~"
-			(at 99.06 68.58 0)
+			(at 99.06 69.85 0)
 			(effects
 				(font
@@
 		)
 		(property "Description" "Unpolarized capacitor"
-			(at 99.06 68.58 0)
+			(at 99.06 69.85 0)
 			(effects
 				(font
@@
 			)
 		)
-		(property "Footprint" ""
+		(property "Footprint" "Capacitor_SMD:C_0402_1005Metric"
 			(at 184.15 76.5048 0)
 			(effects
@@
 			)
 		)
-		(property "Footprint" ""
+		(property "Footprint" "Capacitor_SMD:C_0402_1005Metric"
 			(at 77.1652 63.5 0)
 			(effects
@@
 			)
 		)
-		(property "Footprint" "21-100134_N201A2-1_MXM"
+		(property "Footprint" "Project-Symbols:MAX86140ENP+T"
 			(at 104.14 39.116 0)
 			(effects

Commit message: schematic mostly finished
Parts:
- C17: footprint Capacitor_SMD:C_0402_1005Metric -> Capacitor_SMD:C_01005_0402Metric
Changed lines of the file:
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@@
 			)
 		)
-		(property "Footprint" "Capacitor_SMD:C_0402_1005Metric"
+		(property "Footprint" "Capacitor_SMD:C_01005_0402Metric"
 			(at 89.8652 63.5 0)
 			(effects

Commit message: ready to order
Parts:
- C15: footprint Capacitor_SMD:C_0201_0603Metric -> Capacitor_SMD:C_0603_1608Metric
- C16, C18: footprint Capacitor_SMD:C_0402_1005Metric -> Capacitor_SMD:C_0603_1608Metric
- C17: footprint Capacitor_SMD:C_01005_0402Metric -> Capacitor_SMD:C_0603_1608Metric
Changed lines of the file:
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@@
 			)
 		)
-		(property "Footprint" "Capacitor_SMD:C_01005_0402Metric"
+		(property "Footprint" "Capacitor_SMD:C_0603_1608Metric"
 			(at 89.8652 63.5 0)
 			(effects
@@
 			)
 		)
-		(property "Footprint" "Capacitor_SMD:C_0201_0603Metric"
+		(property "Footprint" "Capacitor_SMD:C_0603_1608Metric"
 			(at 100.0252 73.66 0)
 			(effects
@@
 			)
 		)
-		(property "Footprint" "Capacitor_SMD:C_0402_1005Metric"
+		(property "Footprint" "Capacitor_SMD:C_0603_1608Metric"
 			(at 184.15 76.5048 0)
 			(effects
@@
 			)
 		)
-		(property "Footprint" "Capacitor_SMD:C_0402_1005Metric"
+		(property "Footprint" "Capacitor_SMD:C_0603_1608Metric"
 			(at 77.1652 63.5 0)
 			(effects
