File: accelerometer.kicad_sch (KiCad schematic)
At the start: 4 parts, among them U2 ADXL366BCCZ-RL7

Commit message: General Structure
Other:
- company: (none) -> Guardian Health Inc.
- title: (none) -> ADCL366 Accelerometer
Changed lines of the file:
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@@
 	(generator_version "9.0")
 	(paper "A4")
+	(title_block
+		(title "ADCL366 Accelerometer")
+		(company "Guardian Health Inc.")
+	)
 	(junction
 		(at 88.9 90.17)

Commit message: inital routing
Parts:
- C19, C20, C21: footprint (none) -> Capacitor_SMD:C_01005_0402Metric
- U2: footprint CC-12-4_ADI -> Project-Symbols:ADXL366BCCZ-RL7
Changed lines of the file:
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@@
 			)
 		)
-		(property "Footprint" ""
+		(property "Footprint" "Capacitor_SMD:C_01005_0402Metric"
 			(at 89.8652 87.63 0)
 			(effects
@@
 			)
 		)
-		(property "Footprint" "CC-12-4_ADI"
+		(property "Footprint" "Project-Symbols:ADXL366BCCZ-RL7"
 			(at 111.76 59.69 0)
 			(effects
@@
 			)
 		)
-		(property "Footprint" ""
+		(property "Footprint" "Capacitor_SMD:C_01005_0402Metric"
 			(at 89.8652 97.79 0)
 			(effects
@@
 			)
 		)
-		(property "Footprint" ""
+		(property "Footprint" "Capacitor_SMD:C_01005_0402Metric"
 			(at 180.0352 71.12 0)
 			(effects

Commit message: schematic mostly finished
Connections:
- no-connect marks 0 -> 1
Changed lines of the file:
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@@
 		(color 0 0 0 0)
+	)
+	(no_connect
+		(at 111.76 59.69)
 	)
 	(wire

Commit message: ready to order
Parts:
- C19: footprint Capacitor_SMD:C_01005_0402Metric -> Capacitor_SMD:C_0603_1608Metric
Changed lines of the file:
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@@
 			)
 		)
-		(property "Footprint" "Capacitor_SMD:C_01005_0402Metric"
+		(property "Footprint" "Capacitor_SMD:C_0603_1608Metric"
 			(at 180.0352 71.12 0)
 			(effects

Commit message: resize to 0603
Parts:
- C20, C21: footprint Capacitor_SMD:C_01005_0402Metric -> Capacitor_SMD:C_0603_1608Metric
Changed lines of the file:
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@@
 			)
 		)
-		(property "Footprint" "Capacitor_SMD:C_01005_0402Metric"
+		(property "Footprint" "Capacitor_SMD:C_0603_1608Metric"
 			(at 89.8652 87.63 0)
 			(effects
@@
 			)
 		)
-		(property "Footprint" "Capacitor_SMD:C_01005_0402Metric"
+		(property "Footprint" "Capacitor_SMD:C_0603_1608Metric"
 			(at 89.8652 97.79 0)
 			(effects
