File: health_monitor.kicad_sch (KiCad schematic)
At the start: 0 parts

Commit message: MCU Submodule done
Other:
- added sheet AFE (afe.kicad_sch)
- added sheet MCU (mcu.kicad_sch)

Commit message: schematic 90%
Parts:
- added SENSOR1: SFH7050, SFH7050:OSRAM_SFH7050, symbol ProjectSymbols:SFH7050
Connections:
- new net GNDREF: SENSOR1.4 (PA)
- new net Optical Front-End/LED1_ANODE: SENSOR1.2 (GA)
- new net Optical Front-End/LED1_CATHODE: SENSOR1.1 (GC)
- new net Optical Front-End/LED2_ANODE: SENSOR1.3 (RA)
- new net Optical Front-End/LED2_CATHODE: SENSOR1.6 (RC)
- new net Optical Front-End/LED3_ANODE: SENSOR1.7 (IA)
- new net Optical Front-End/LED3_CATHODE: SENSOR1.8 (IC)
- new net Optical Front-End/PD1: SENSOR1.5 (PC)
Other:
- sheet AFE renamed Optical Front-End
- sheet MCU renamed Microcontroller
- added sheet Accelerometer (accelerometer.kicad_sch)
- added sheet Power Management (power.kicad_sch)
- sheet Microcontroller ports: added DIO_16, DIO_17, JTAG_TCKC, JTAG_TMSC; removed DIO_6, JTAG-TCKC, JTAG-TMSC
- sheet Optical Front-End ports: added GND, GPIO1, GPIO2, INT, LED1_ANODE, LED1_CATHODE, LED2_ANODE, LED2_CATHODE, LED3_ANODE, LED3_CATHODE, PD1, PD_GND, SPI_CSB, SPI_SCLK, SPI_SDI, SPI_SDO, VDD_ANALOG, VDD_DIGITAL, VDD_LED; removed none
- company: (none) -> Guardian Health Inc.
- title: (none) -> Wearable Vital Monitor

Commit message: General Structure
Connections:
- net MAX86140 AFE/LED1_ANODE renamed LED_ANODE0
- net MAX86140 AFE/LED1_CATHODE renamed LED_CATHODE0
- net MAX86140 AFE/LED2_ANODE renamed LED_ANODE1
- net MAX86140 AFE/LED2_CATHODE renamed LED_CATHODE1
- net MAX86140 AFE/LED3_ANODE renamed LED_ANODE2
- net MAX86140 AFE/LED3_CATHODE renamed LED_CATHODE2
- net MAX86140 AFE/PD1 renamed PD1
Other:
- sheet Optical Front-End renamed MAX86140 AFE
- sheet MAX86140 AFE ports: added ANALOG_GND, LED_ANODE[0..2], LED_CATHODE[0..2], LED_GND; removed LED1_ANODE, LED1_CATHODE, LED2_ANODE, LED2_CATHODE, LED3_ANODE, LED3_CATHODE
- sheet Microcontroller ports: added DIO[0..30]; removed DIO_0, DIO_1, DIO_10, DIO_11, DIO_12, DIO_13, DIO_16, DIO_17, DIO_2, DIO_3, DIO_4, DIO_5, DIO_7, DIO_8, DIO_9
- sheet Power Management ports: added BAT, CHG_VDD, INT, MPC[0..7], SCL, SDA; removed none

Commit message: inital routing
Parts:
- added J1: USBC, Project-Symbols:CONN16_203615_MOL, symbol ProjectSymbols:USBC
- added J2: BAT+_PAD, Connector_PinHeader_2.54mm:PinHeader_1x01_P2.54mm_Vertical, symbol Connector:Conn_01x01_Pin
- added J3: THERMISTOR, Connector_PinHeader_2.54mm:PinHeader_1x02_P2.54mm_Vertical, symbol Connector:Screw_Terminal_01x02
- added J4: JTAG_HEADER, Connector_PinHeader_2.54mm:PinHeader_1x06_P2.54mm_Vertical, symbol Connector:Conn_ARM_JTAG_SWD_10
- added J5: RFP_PAD, Connector_PinHeader_2.54mm:PinHeader_1x01_P2.54mm_Vertical, symbol Connector:Conn_01x01_Pin
- added J6: RFN_PAD, Connector_PinHeader_2.54mm:PinHeader_1x01_P2.54mm_Vertical, symbol Connector:Conn_01x01_Pin
- SENSOR1: footprint SFH7050:OSRAM_SFH7050 -> Project-Symbols:SFH 7050A_OSM
Connections:
- net GNDREF: now also J1.A1 (GND), J1.A12 (GND), J1.B1 (GND), J1.B12 (GND), J1.GND1, J1.GND2, J3.2 (Pin_2), J4.3 (GND), J4.5 (GND), J4.9 (GNDDetect)
- net CC2674R10/RESET: now also J4.10 (~{RESET})
- new net CC1: J1.A5 (CC_{1})
- new net CC2: J1.B5 (CC_{2})
- new net CC2674R10/JTAG_{TCKC}: J4.4 (SWCLK/TCK)
- new net CC2674R10/JTAG_{TMSC}: J4.2 (SWDIO/TMS)
- new net CC2674R10/RF_{N}: J6.1 (Pin_1)
- new net CC2674R10/RF_{P}: J5.1 (Pin_1)
- new net MCU_DIO16: J4.6 (SWO/TDO)
- new net MCU_DIO17: J4.8 (NC/TDI)
- new net Power Management ICs/BAT+: J2.1 (Pin_1)
- new net Power Management ICs/DN: J1.A7 (D_{-}), J1.B7 (D_{-})
- new net Power Management ICs/DP: J1.A6 (D_{+}), J1.B6 (D_{+})
- new net Power Management ICs/THM+: J3.1 (Pin_1)
- new net V_{BUS}: J1.A4 (V_{BUS}), J1.A9 (V_{BUS}), J1.B4 (V_{BUS}), J1.B9 (V_{BUS})
- new net V_{D}: J4.1 (VTref)
- no-connect marks 0 -> 2
Other:
- sheet Microcontroller renamed CC2674R10
- sheet Power Management renamed Power Management ICs
- sheet CC2674R10 ports: added JTAG_{TCKC}, JTAG_{TMSC}, RF_{N}, RF_{P}, V_{DD}; removed JTAG_TCKC, JTAG_TMSC, RF_N, RF_P, VDD
- sheet Power Management ICs ports: added BAT+, CC1, CC2, CHG_EN, CHG_INT, CHG_SCL, CHG_SDA, DN, DP, THM+, V_{2.0}, V_{ANALOG}, V_{BUS}, V_{DIGITAL}, V_{LED}; removed ACCEL_VDD_ANALOG, ACCEL_VDD_DIGITAL, AFE_VDD_ANALOG, AFE_VDD_DIGITAL, AFE_VDD_LED, BAT, CHG_VDD, INT, MCU_VDD, MPC[0..7], SCL, SDA
- moved on the sheet: SENSOR1

Commit message: schematic mostly finished
Parts:
- removed J2: BAT+_PAD, Connector_PinHeader_2.54mm:PinHeader_1x01_P2.54mm_Vertical, symbol Connector:Conn_01x01_Pin
- removed J3: THERMISTOR, Connector_PinHeader_2.54mm:PinHeader_1x02_P2.54mm_Vertical, symbol Connector:Screw_Terminal_01x02
- removed J4: JTAG_HEADER, Connector_PinHeader_2.54mm:PinHeader_1x06_P2.54mm_Vertical, symbol Connector:Conn_ARM_JTAG_SWD_10
- removed J5: RFP_PAD, Connector_PinHeader_2.54mm:PinHeader_1x01_P2.54mm_Vertical, symbol Connector:Conn_01x01_Pin
- removed J6: RFN_PAD, Connector_PinHeader_2.54mm:PinHeader_1x01_P2.54mm_Vertical, symbol Connector:Conn_01x01_Pin
- added AE1: Antenna, RF_Antenna:Johanson_2450AT18x100, symbol Device:Antenna
- added C32: 1pF, Capacitor_SMD:C_0402_1005Metric, symbol Device:C_Small
- added J2: Conn_01x02_Pin, Connector_PinHeader_2.54mm:PinHeader_1x02_P2.54mm_Vertical, symbol Connector:Conn_01x02_Pin
- added J3: Conn_01x05, Connector_PinHeader_2.54mm:PinHeader_1x05_P2.54mm_Vertical, symbol Connector_Generic:Conn_01x05
- added L3: 3.9nH, Inductor_SMD:L_0402_1005Metric, symbol Device:L_Small
- added L4: 2.7nH, Inductor_SMD:L_0402_1005Metric, symbol Device:L_Small
Connections:
- net CC2674R10/JTAG_{TCKC}: now also J3.1 (Pin_1)
- net CC2674R10/JTAG_{TMSC}: now also J3.2 (Pin_2)
- net CC2674R10/RESET: now also J3.5 (Pin_5)
- net CC2674R10/RF_{P}: now also C32.1
- net GNDREF: now also J2.2 (Pin_2), L4.2
- net MCU_DIO16: now also J3.3 (Pin_3)
- net MCU_DIO17: now also J3.4 (Pin_4)
- net Power Management ICs/BAT+: now also J2.1 (Pin_1)
- net CC1: no longer names the net of J1.A5 (CC_{1})
- net CC2: no longer names the net of J1.B5 (CC_{2})
- net Power Management ICs/DN: no longer names the net of J1.A7 (D_{-})
- net Power Management ICs/DN: no longer J1.B7 (D_{-})
- net Power Management ICs/DP: no longer names the net of J1.A6 (D_{+})
- net Power Management ICs/DP: no longer J1.B6 (D_{+})
- new net: C32.2, L3.1, L4.1
- new net: AE1.1 (A), L3.2
- no-connect marks 2 -> 11
Other:
- sheet Power Management ICs ports: added none; removed CC1, CC2, CHG_EN, CHG_INT, DN, DP, THM+, V_{DIGITAL}

Commit message: ready to order
Parts:
- AE1: LCSC PN (none) -> C161362
- J1: footprint Project-Symbols:CONN16_203615_MOL -> Project-Symbols:MOLEX_USBC_1054500101; LCSC PN (none) -> C5447355
Changed lines of the file:
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@@
+			)
+		)
+		(property "LCSC PN" "C161362"
+			(at 255.27 59.69 0)
+			(effects
+				(font
+					(size 1.27 1.27)
+				)
+				(hide yes)
 			)
 		)
@@
 			)
 		)
-		(property "Footprint" "Project-Symbols:CONN16_203615_MOL"
+		(property "Footprint" "Project-Symbols:MOLEX_USBC_1054500101"
 			(at 36.322 14.986 0)
 			(effects
@@
 			(at 29.21 31.75 0)
 			(effects
+				(font
+					(size 1.27 1.27)
+				)
+				(hide yes)
+			)
+		)
+		(property "LCSC PN" "C5447355"
+			(at 29.21 31.75 0)
+			(effects

Commit message: resize to 0603
Parts:
- C32: footprint Capacitor_SMD:C_0402_1005Metric -> Capacitor_SMD:C_0603_1608Metric
- L3, L4: footprint Inductor_SMD:L_0402_1005Metric -> Inductor_SMD:L_0603_1608Metric
Changed lines of the file:
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@@
 			)
 		)
-		(property "Footprint" "Inductor_SMD:L_0402_1005Metric"
+		(property "Footprint" "Inductor_SMD:L_0603_1608Metric"
 			(at 241.3 69.85 0)
 			(effects
@@
 			)
 		)
-		(property "Footprint" "Capacitor_SMD:C_0402_1005Metric"
+		(property "Footprint" "Capacitor_SMD:C_0603_1608Metric"
 			(at 236.22 66.04 0)
 			(effects
@@
 			)
 		)
-		(property "Footprint" "Inductor_SMD:L_0402_1005Metric"
+		(property "Footprint" "Inductor_SMD:L_0603_1608Metric"
 			(at 248.92 66.04 0)
 			(effects

Commit message: final order
Parts:
- AE1: LCSC PN C161362 -> C89334
- J1: LCSC PN C5447355 -> C134092
Changed lines of the file:
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@@
 			)
 		)
-		(property "LCSC PN" "C161362"
+		(property "LCSC PN" "C89334"
 			(at 255.27 59.69 0)
 			(effects
@@
 			)
 		)
-		(property "LCSC PN" "C5447355"
+		(property "LCSC PN" "C134092"
 			(at 29.21 31.75 0)
 			(effects
