File: mcu.kicad_sch (KiCad schematic)
At the start: 14 parts

Commit message: schematic 90%
Parts:
- removed C3: 10uF, Capacitor_SMD:C_0805_2012Metric, symbol Device:C
- removed FC-135-1: 32.768kHz, XTAL_FC-135_EPS, symbol ProjectSymbols:FC-135_32.7680KA-A5
- removed MCU0: CC2640R2FYFVR, YFV0034ALAL, symbol ProjectSymbols:CC2640R2FYFVR
- removed TSX-150-1: 24MHz, symbol ProjectSymbols:TSX-3225
- added C11, C12, C13, C14: 10pF, Capacitor_SMD:C_1206_3216Metric, symbol Device:C
- added C5: 100nF, Capacitor_SMD:C_1206_3216Metric, symbol Device:C
- added C6: 22uF, Capacitor_SMD:C_0805_2012Metric, symbol Device:C
- added CX2016FB-1: 48MHz, Crystal:Crystal_SMD_2016-4Pin_2.0x1.6mm, symbol Device:Crystal_GND24
- added MCU1: CC2674R106T0RGZR, VQFN48_RGZ_TEX, symbol ProjectSymbols:CC2674R106T0RGZR
- added NX2012SA-1: 32.768 kHz, Crystal:Crystal_SMD_2012-2Pin_2.0x1.2mm, symbol ProjectSymbols:FC-135_32.7680KA-A5
- C4: value 10uF -> 22uF
- C9: value 10uF -> 100nF; footprint Capacitor_SMD:C_0805_2012Metric -> Capacitor_SMD:C_1206_3216Metric
- L1: value 10uF -> 6.8uH
- renumbered C8 to C10, C5 to C3, C6 to C8
Connections:
- net DIO_0: now also MCU1.5 (DIO_0)
- net DIO_1: now also MCU1.6 (DIO_1)
- net DIO_10: now also MCU1.16 (DIO_10)
- net DIO_11: now also MCU1.17 (DIO_11)
- net DIO_12: now also MCU1.18 (DIO_12)
- net DIO_13: now also MCU1.19 (DIO_13)
- net DIO_2: now also MCU1.7 (DIO_2)
- net DIO_3: now also MCU1.8 (DIO_3)
- net DIO_4: now also MCU1.9 (DIO_4)
- net DIO_5: now also MCU1.10 (DIO_5)
- net DIO_6: now also MCU1.11 (DIO_6)
- net DIO_7: now also MCU1.12 (DIO_7)
- net DIO_8: now also MCU1.14 (DIO_8)
- net DIO_9: now also MCU1.15 (DIO_9)
- net GND: now also C3.2, C4.1, C7.2, C9.2, C11.2, C12.1, C13.2, C14.1, C5.2, C6.1, CX2016FB-1.2, CX2016FB-1.4, MCU1.49 (EGP); no longer C3.1, C4.2, C7.1, C9.1
- net RESET: now also MCU1.35 (RESET_N)
- net RF_N: now also MCU1.2 (RF_N_2_4GHZ)
- net RF_P: now also MCU1.1 (RF_P_2_4GHZ)
- net VDD: now also C3.1, C4.2, C5.1, MCU1.13 (VDDS2), MCU1.22 (VDDS3), MCU1.34 (VDDS_DCDC), MCU1.44 (VDDS); no longer C3.2, C4.1
- net at C8.1, L1.1: now also C7.1, C6.2, MCU1.45 (VDDR), MCU1.48 (VDDR_RF); no longer C7.2
- net at L1.2: now also MCU1.33 (DCDC_SW)
- new net: C14.2, CX2016FB-1.1, MCU1.46 (X48M_N)
- new net: C13.1, CX2016FB-1.3, MCU1.47 (X48M_P)
- new net: C12.2, MCU1.4 (K32X_Q2), NX2012SA-1.1
- new net: C9.1, MCU1.23 (DCOUPL)
- new net: C11.1, MCU1.3 (K32X_Q1), NX2012SA-1.2
- new net DIO_14: MCU1.20 (DIO_14)
- new net DIO_15: MCU1.21 (DIO_15)
- new net DIO_16: MCU1.26 (DIO_16)
- new net DIO_17: MCU1.27 (DIO_17)
- new net DIO_18: MCU1.28 (DIO_18)
- new net DIO_19: MCU1.29 (DIO_19)
- new net DIO_20: MCU1.30 (DIO_20)
- new net DIO_21: MCU1.31 (DIO_21)
- new net DIO_22: MCU1.32 (DIO_22)
- new net DIO_23: MCU1.36 (DIO_23)
- new net DIO_24: MCU1.37 (DIO_24)
- new net DIO_25: MCU1.38 (DIO_25)
- new net DIO_26: MCU1.39 (DIO_26)
- new net DIO_27: MCU1.40 (DIO_27)
- new net DIO_28: MCU1.41 (DIO_28)
- new net DIO_29: MCU1.42 (DIO_29)
- new net DIO_30: MCU1.43 (DIO_30)
- new net JTAG_TCKC: MCU1.24 (JTAG_TMSC)
- new net JTAG_TMSC: MCU1.25 (JTAG_TCKC)
Other:
- moved on the sheet: C1, C10, C2, C3, C4, C7, C8, L1, R1

Commit message: General Structure
Connections:
- net DIO_0 renamed DIO0
- net DIO_1 renamed DIO1
- net DIO_10 renamed DIO10
- net DIO_11 renamed DIO11
- net DIO_12 renamed DIO12
- net DIO_13 renamed DIO13
- net DIO_14 renamed DIO14
- net DIO_15 renamed DIO15
- net DIO_16 renamed DIO16
- net DIO_17 renamed DIO17
- net DIO_18 renamed DIO18
- net DIO_19 renamed DIO19
- net DIO_2 renamed DIO2
- net DIO_20 renamed DIO20
- net DIO_21 renamed DIO21
- net DIO_22 renamed DIO22
- net DIO_23 renamed DIO23
- net DIO_24 renamed DIO24
- net DIO_25 renamed DIO25
- net DIO_26 renamed DIO26
- net DIO_27 renamed DIO27
- net DIO_28 renamed DIO28
- net DIO_29 renamed DIO29
- net DIO_3 renamed DIO3
- net DIO_30 renamed DIO30
- net DIO_4 renamed DIO4
- net DIO_5 renamed DIO5
- net DIO_6 renamed DIO6
- net DIO_7 renamed DIO7
- net DIO_8 renamed DIO8
- net DIO_9 renamed DIO9
Other:
- company: (none) -> Guardian Health Inc.
- title: MCU -> CC2674R10 Microcontroller

Commit message: inital routing
Parts:
- C1, C10, C11, C12, C13, C14, C2, C3, C5, C7, C8, C9: footprint Capacitor_SMD:C_1206_3216Metric -> Capacitor_SMD:C_01005_0402Metric
- C4, C6: footprint Capacitor_SMD:C_0805_2012Metric -> Capacitor_SMD:C_0402_1005Metric
- L1: footprint (none) -> Inductor_SMD:L_Pulse_PA4332; MouserURL (none) -> https://www.mouser.com/ProductDetail/Pulse-Electronics/PA43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
- MCU1: footprint VQFN48_RGZ_TEX -> Project-Symbols:CC2647R106T0RGZR
- R1: footprint (none) -> Resistor_SMD:R_0603_1608Metric
Connections:
- net JTAG_TCKC renamed JTAG_{TCKC}
- net JTAG_TMSC renamed JTAG_{TMSC}
- net RF_N renamed RF_{N}
- net RF_P renamed RF_{P}
- net VDD renamed V_{DD}
Changed lines of the file:
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@@
 	)
 	(hierarchical_label "GND"
-		(shape input)
+		(shape passive)
 		(at 104.14 73.66 180)
 		(effects
@@
 	)
 	(hierarchical_label "GND"
-		(shape input)
+		(shape passive)
 		(at 123.19 48.26 180)
 		(effects
@@
 	)
 	(hierarchical_label "GND"
-		(shape input)
+		(shape passive)
 		(at 116.84 66.04 180)
 		(effects
@@
 	)
 	(hierarchical_label "GND"
-		(shape input)
+		(shape passive)
 		(at 78.74 137.16 270)
 		(effects
@@
 		)
 	)
-	(hierarchical_label "RF_P"
+	(hierarchical_label "RF_{P}"
 		(shape bidirectional)
 		(at 144.78 129.54 180)
@@
 	)
 	(hierarchical_label "GND"
-		(shape input)
+		(shape passive)
 		(at 123.19 85.09 180)
 		(effects
@@
 		)
 	)
-	(hierarchical_label "JTAG_TCKC"
+	(hierarchical_label "JTAG_{TCKC}"
 		(shape input)
 		(at 144.78 118.11 180)
@@
 	)
 	(hierarchical_label "GND"
-		(shape input)
+		(shape passive)
 		(at 90.17 92.71 180)
 		(effects
@@
 	)
 	(hierarchical_label "GND"
-		(shape input)
+		(shape passive)
 		(at 128.27 128.27 0)
 		(effects
@@
 	)
 	(hierarchical_label "GND"
-		(shape input)
+		(shape passive)
 		(at 73.66 121.92 180)
 		(effects
@@
 	)
 	(hierarchical_label "GND"
-		(shape input)
+		(shape passive)
 		(at 105.41 88.9 180)
 		(effects
@@
 	)
 	(hierarchical_label "GND"
-		(shape input)
+		(shape passive)
 		(at 123.19 99.06 180)
 		(effects
@@
 		)
 	)
-	(hierarchical_label "VDD"
+	(hierarchical_label "V_{DD}"
 		(shape input)
 		(at 101.6 128.27 180)
@@
 	)
 	(hierarchical_label "GND"
-		(shape input)
+		(shape passive)
 		(at 78.74 105.41 90)
 		(effects
@@
 	)
 	(hierarchical_label "GND"
-		(shape input)
+		(shape passive)
 		(at 83.82 121.92 0)
 		(effects
@@
 	)
 	(hierarchical_label "GND"
-		(shape input)
+		(shape passive)
 		(at 110.49 52.07 180)
 		(effects
@@
 		)
 	)
-	(hierarchical_label "RF_N"
+	(hierarchical_label "RF_{N}"
 		(shape bidirectional)
 		(at 144.78 132.08 180)
@@
 	)
 	(hierarchical_label "GND"
-		(shape input)
+		(shape passive)
 		(at 135.89 44.45 180)
 		(effects
@@
 	)
 	(hierarchical_label "GND"
-		(shape input)
+		(shape passive)
 		(at 129.54 62.23 180)
 		(effects
@@
 		)
 	)
-	(hierarchical_label "VDD"
+	(hierarchical_label "V_{DD}"
 		(shape input)
 		(at 147.32 44.45 0)
@@
 		)
 	)
-	(hierarchical_label "JTAG_TMSC"
+	(hierarchical_label "JTAG_{TMSC}"
 		(shape input)
 		(at 144.78 120.65 180)
@@
 	)
 	(hierarchical_label "DIO[0..30]"
-		(shape input)
+		(shape bidirectional)
 		(at 228.6 139.7 0)
 		(effects
@@
 			)
 		)
-		(property "Footprint" "Capacitor_SMD:C_1206_3216Metric"
+		(property "Footprint" "Capacitor_SMD:C_01005_0402Metric"
 			(at 105.41 89.8652 0)
 			(effects
@@
 			)
 		)
-		(property "Footprint" "Capacitor_SMD:C_0805_2012Metric"
+		(property "Footprint" "Capacitor_SMD:C_0402_1005Metric"
 			(at 111.76 72.6948 0)
 			(effects
@@
 			)
 		)
-		(property "Footprint" ""
+		(property "Footprint" "Inductor_SMD:L_Pulse_PA4332"
 			(at 135.89 73.66 0)
 			(effects
@@
 		(property "Description" "Inductor"
 			(at 135.89 73.66 0)
+			(effects
+				(font
+					(size 1.27 1.27)
+				)
+				(hide yes)
+			)
+		)
+		(property "MouserURL" "https://www.mouser.com/ProductDetail/Pulse-Electronics/PA4332.682NLT?qs=%2FzQKu7YvIMbRulhkYYDqtA%3D%3D"
+			(at 135.89 73.66 90)
 			(effects
 				(font
@@
 			)
 		)
-		(property "Footprint" "Capacitor_SMD:C_1206_3216Metric"
+		(property "Footprint" "Capacitor_SMD:C_01005_0402Metric"
 			(at 79.7052 113.03 0)
 			(effects
@@
 			)
 		)
-		(property "Footprint" "Capacitor_SMD:C_1206_3216Metric"
+		(property "Footprint" "Capacitor_SMD:C_01005_0402Metric"
 			(at 123.19 86.0552 0)
 			(effects
@@
 			)
 		)
-		(property "Footprint" "Capacitor_SMD:C_1206_3216Metric"
+		(property "Footprint" "Capacitor_SMD:C_01005_0402Metric"
 			(at 135.89 45.4152 0)
 			(effects
@@
 			)
 		)
-		(property "Footprint" "Capacitor_SMD:C_1206_3216Metric"
+		(property "Footprint" "Capacitor_SMD:C_01005_0402Metric"
 			(at 123.19 49.2252 0)
 			(effects
@@
 			)
 		)
-		(property "Footprint" "Capacitor_SMD:C_1206_3216Metric"
+		(property "Footprint" "Capacitor_SMD:C_01005_0402Metric"
 			(at 125.73 127.3048 0)
 			(effects
@@
 			)
 		)
-		(property "Footprint" "Capacitor_SMD:C_1206_3216Metric"
+		(property "Footprint" "Capacitor_SMD:C_01005_0402Metric"
 			(at 97.79 105.7148 0)
 			(effects
@@
 			)
 		)
-		(property "Footprint" "Capacitor_SMD:C_1206_3216Metric"
+		(property "Footprint" "Capacitor_SMD:C_01005_0402Metric"
 			(at 79.7052 137.16 0)
 			(effects
@@
 			)
 		)
-		(property "Footprint" ""
+		(property "Footprint" "Resistor_SMD:R_0603_1608Metric"
 			(at 107.95 130.048 90)
 			(effects
@@
 			)
 		)
-		(property "Footprint" "Capacitor_SMD:C_1206_3216Metric"
+		(property "Footprint" "Capacitor_SMD:C_01005_0402Metric"
 			(at 110.49 53.0352 0)
 			(effects
@@
 			)
 		)
-		(property "Footprint" "VQFN48_RGZ_TEX"
+		(property "Footprint" "Project-Symbols:CC2647R106T0RGZR"
 			(at 146.05 37.084 0)
 			(effects
@@
 			)
 		)
-		(property "Footprint" "Capacitor_SMD:C_1206_3216Metric"
+		(property "Footprint" "Capacitor_SMD:C_01005_0402Metric"
 			(at 90.17 93.6752 0)
 			(effects
@@
 			)
 		)
-		(property "Footprint" "Capacitor_SMD:C_1206_3216Metric"
+		(property "Footprint" "Capacitor_SMD:C_01005_0402Metric"
 			(at 123.19 100.0252 0)
 			(effects
@@
 			)
 		)
-		(property "Footprint" "Capacitor_SMD:C_0805_2012Metric"
+		(property "Footprint" "Capacitor_SMD:C_0402_1005Metric"
 			(at 137.16 61.2648 0)
 			(effects
@@
 			)
 		)
-		(property "Footprint" "Capacitor_SMD:C_1206_3216Metric"
+		(property "Footprint" "Capacitor_SMD:C_01005_0402Metric"
 			(at 116.84 67.0052 0)
 			(effects

Commit message: schematic mostly finished
Parts:
- removed L1: 6.8uH, Inductor_SMD:L_Pulse_PA4332, symbol Device:L
- R1: footprint Resistor_SMD:R_0603_1608Metric -> Resistor_SMD:R_0402_1005Metric_Pad0.72x0.64mm_HandSolder
Connections:
- no-connect marks 0 -> 1
Changed lines of the file:
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@@
-	)
-	(junction
-		(at 130.81 73.66)
-		(diameter 0)
-		(color 0 0 0 0)
 	)
 	(junction
@@
 		(color 0 0 0 0)
 	)
+	(no_connect
+		(at 144.78 78.74)
+	)
 	(bus_entry
 		(at 213.36 86.36)
@@
 	(wire
 		(pts
-			(xy 142.24 78.74) (xy 144.78 78.74)
-		)
-		(stroke
-			(width 0)
-			(type default)
-		)
-	)
-	(wire
-		(pts
 			(xy 205.74 60.96) (xy 213.36 60.96)
 		)
@@
 	(wire
 		(pts
-			(xy 130.81 73.66) (xy 132.08 73.66)
-		)
-		(stroke
-			(width 0)
-			(type default)
-		)
-	)
-	(wire
-		(pts
 			(xy 139.7 62.23) (xy 137.16 62.23)
 		)
@@
 	(wire
 		(pts
-			(xy 142.24 73.66) (xy 142.24 78.74)
-		)
-		(stroke
-			(width 0)
-			(type default)
-		)
-	)
-	(wire
-		(pts
 			(xy 205.74 91.44) (xy 213.36 91.44)
 		)
@@
 		(pts
 			(xy 215.9 78.74) (xy 215.9 81.28)
-		)
-		(stroke
-			(width 0)
-			(type default)
-		)
-	)
-	(wire
-		(pts
-			(xy 139.7 73.66) (xy 142.24 73.66)
 		)
 		(stroke
@@
 			)
 		)
-		(property "Description" "Four pin crystal, GND on pins 2 and 4; CX2016FB48000D0FZZH1"
+		(property "Description" "Four pin crystal, GND on pins 2 and 4; NX2016SA-48MHZ-EXS00A-CS05517"
 			(at 78.74 121.92 0)
 			(effects
@@
 				(path "/c6abb77c-95da-4337-b8bb-663a91b271f5/0600b84d-9564-4910-a69f-e5ec417d5f8b"
 					(reference "CX2016FB-1")
-					(unit 1)
-				)
-			)
-		)
-	)
-	(symbol
-		(lib_id "Device:L")
-		(at 135.89 73.66 90)
-		(unit 1)
-		(exclude_from_sim no)
-		(in_bom yes)
-		(on_board yes)
-		(dnp no)
-		(property "Reference" "L1"
-			(at 135.89 68.58 90)
-			(effects
-				(font
-					(size 1.27 1.27)
-				)
-			)
-		)
-		(property "Value" "6.8uH"
-			(at 135.89 71.12 90)
-			(effects
-				(font
-					(size 1.27 1.27)
-				)
-			)
-		)
-		(property "Footprint" "Inductor_SMD:L_Pulse_PA4332"
-			(at 135.89 73.66 0)
-			(effects
-				(font
-					(size 1.27 1.27)
-				)
-				(hide yes)
-			)
-		)
-		(property "Datasheet" "~"
-			(at 135.89 73.66 0)
-			(effects
-				(font
-					(size 1.27 1.27)
-				)
-				(hide yes)
-			)
-		)
-		(property "Description" "Inductor"
-			(at 135.89 73.66 0)
-			(effects
-				(font
-					(size 1.27 1.27)
-				)
-				(hide yes)
-			)
-		)
-		(property "MouserURL" "https://www.mouser.com/ProductDetail/Pulse-Electronics/PA4332.682NLT?qs=%2FzQKu7YvIMbRulhkYYDqtA%3D%3D"
-			(at 135.89 73.66 90)
-			(effects
-				(font
-					(size 1.27 1.27)
-				)
-				(hide yes)
-			)
-		)
-		(pin "1"
-		)
-		(pin "2"
-		)
-		(instances
-			(project "health_monitor"
-				(path "/c6abb77c-95da-4337-b8bb-663a91b271f5/0600b84d-9564-4910-a69f-e5ec417d5f8b"
-					(reference "L1")
-					(unit 1)
-				)
-			)
-			(project ""
-				(path "/e9ed16af-9ab2-4ec3-95b1-0b878a10626b"
-					(reference "L1")
 					(unit 1)
 				)
@@
 			)
 		)
-		(property "Footprint" "Resistor_SMD:R_0603_1608Metric"
+		(property "Footprint" "Resistor_SMD:R_0402_1005Metric_Pad0.72x0.64mm_HandSolder"
 			(at 107.95 130.048 90)
 			(effects
@@
 			)
 		)
-		(property "Description" ""
+		(property "Description" "NX2012SA-32.768KHZ-STD-MUB-2"
 			(at 104.14 104.14 0)
 			(effects

Commit message: resize to 0603
Parts:
- C1, C11, C12, C13, C14, C2, C3, C5, C7, C8, C9: footprint Capacitor_SMD:C_01005_0402Metric -> Capacitor_SMD:C_0603_1608Metric
- C10: footprint Capacitor_SMD:C_01005_0402Metric -> Capacitor_SMD:C_0603_1608Metric_Pad1.08x0.95mm_HandSolder
- C4, C6: footprint Capacitor_SMD:C_0402_1005Metric -> Capacitor_SMD:C_0603_1608Metric
- R1: footprint Resistor_SMD:R_0402_1005Metric_Pad0.72x0.64mm_HandSolder -> Resistor_SMD:R_0603_1608Metric
Changed lines of the file:
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@@
 			)
 		)
-		(property "Footprint" "Capacitor_SMD:C_01005_0402Metric"
+		(property "Footprint" "Capacitor_SMD:C_0603_1608Metric"
 			(at 105.41 89.8652 0)
 			(effects
@@
 			)
 		)
-		(property "Footprint" "Capacitor_SMD:C_0402_1005Metric"
+		(property "Footprint" "Capacitor_SMD:C_0603_1608Metric"
 			(at 111.76 72.6948 0)
 			(effects
@@
 			)
 		)
-		(property "Footprint" "Capacitor_SMD:C_01005_0402Metric"
+		(property "Footprint" "Capacitor_SMD:C_0603_1608Metric"
 			(at 79.7052 113.03 0)
 			(effects
@@
 			)
 		)
-		(property "Footprint" "Capacitor_SMD:C_01005_0402Metric"
+		(property "Footprint" "Capacitor_SMD:C_0603_1608Metric"
 			(at 123.19 86.0552 0)
 			(effects
@@
 			)
 		)
-		(property "Footprint" "Capacitor_SMD:C_01005_0402Metric"
+		(property "Footprint" "Capacitor_SMD:C_0603_1608Metric"
 			(at 135.89 45.4152 0)
 			(effects
@@
 			)
 		)
-		(property "Footprint" "Capacitor_SMD:C_01005_0402Metric"
+		(property "Footprint" "Capacitor_SMD:C_0603_1608Metric"
 			(at 123.19 49.2252 0)
 			(effects
@@
 			)
 		)
-		(property "Footprint" "Capacitor_SMD:C_01005_0402Metric"
+		(property "Footprint" "Capacitor_SMD:C_0603_1608Metric_Pad1.08x0.95mm_HandSolder"
 			(at 125.73 127.3048 0)
 			(effects
@@
 			)
 		)
-		(property "Footprint" "Capacitor_SMD:C_01005_0402Metric"
+		(property "Footprint" "Capacitor_SMD:C_0603_1608Metric"
 			(at 97.79 105.7148 0)
 			(effects
@@
 			)
 		)
-		(property "Footprint" "Capacitor_SMD:C_01005_0402Metric"
+		(property "Footprint" "Capacitor_SMD:C_0603_1608Metric"
 			(at 79.7052 137.16 0)
 			(effects
@@
 			)
 		)
-		(property "Footprint" "Resistor_SMD:R_0402_1005Metric_Pad0.72x0.64mm_HandSolder"
+		(property "Footprint" "Resistor_SMD:R_0603_1608Metric"
 			(at 107.95 130.048 90)
 			(effects
@@
 			)
 		)
-		(property "Footprint" "Capacitor_SMD:C_01005_0402Metric"
+		(property "Footprint" "Capacitor_SMD:C_0603_1608Metric"
 			(at 110.49 53.0352 0)
 			(effects
@@
 			)
 		)
-		(property "Footprint" "Capacitor_SMD:C_01005_0402Metric"
+		(property "Footprint" "Capacitor_SMD:C_0603_1608Metric"
 			(at 90.17 93.6752 0)
 			(effects
@@
 			)
 		)
-		(property "Footprint" "Capacitor_SMD:C_01005_0402Metric"
+		(property "Footprint" "Capacitor_SMD:C_0603_1608Metric"
 			(at 123.19 100.0252 0)
 			(effects
@@
 			)
 		)
-		(property "Footprint" "Capacitor_SMD:C_0402_1005Metric"
+		(property "Footprint" "Capacitor_SMD:C_0603_1608Metric"
 			(at 137.16 61.2648 0)
 			(effects
@@
 			)
 		)
-		(property "Footprint" "Capacitor_SMD:C_01005_0402Metric"
+		(property "Footprint" "Capacitor_SMD:C_0603_1608Metric"
 			(at 116.84 67.0052 0)
 			(effects

Commit message: final order
Parts:
- CX2016FB-1: LCSC PN (none) -> C5186571
- NX2012SA-1: LCSC PN (none) -> C891748
Changed lines of the file:
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@@
+			)
+		)
+		(property "LCSC PN" "C5186571"
+			(at 78.74 121.92 90)
+			(effects
+				(font
+					(size 1.27 1.27)
+				)
+				(hide yes)
 			)
 		)
@@
 			(effects
 				(font
+					(size 1.27 1.27)
+				)
+				(hide yes)
+			)
+		)
+		(property "LCSC PN" "C891748"
+			(at 104.14 104.14 90)
+			(effects
+				(font
